Commit message: gazebo done

File: bot_description/install/bot_description/share/bot_description/urdf/bot_base.urdf (robot description, URDF)
Before this commit: robot my_car, 8 links, 7 joints
Links:
- added link LiDAR, mass 5.0; collision cylinder length=0.08 radius=0.1; visual cylinder length=0.08 radius=0.1
- link front_left_roll: mass None -> 5.0; geometry collision cylinder length=0.1 radius=0.12; visual cylinder length=0.1 radius=0.12
- link front_left_wheel: geometry visual cylinder length=0.1 radius=0.12
- link front_right_roll: mass None -> 5.0; geometry collision cylinder length=0.1 radius=0.12; visual cylinder length=0.1 radius=0.12
- link front_right_wheel: geometry visual cylinder length=0.1 radius=0.12
- link rear_left_wheel: mass None -> 5.0; geometry collision cylinder length=0.1 radius=0.12; visual cylinder length=0.1 radius=0.12
- link rear_right_wheel: mass None -> 5.0; geometry collision cylinder length=0.1 radius=0.12; visual cylinder length=0.1 radius=0.12
Joints:
- added joint LiDAR_joint: type fixed, parent base, child LiDAR, origin xyz=0.22 0 0.13 rpy=0.0 0.0 0.0, axis 0.0 0.0 0.0
